File: 8259.sch (KiCad schematic (older format))
At the start: 11 parts, among them SW23 SW_Push

Commit message: Fixing Weirdness
Parts:
- removed C31: .00001, symbol Device:C
- removed R14: 10000, symbol Device:R
- added C43: 10uF, symbol Device:C
- added D10: DIODE, symbol pspice:DIODE
- added R31: 10k, symbol Device:R
- C41, C42, C44: renamed from C?; value .0000001 -> 0.1uF
- J3: renamed from J?; value Conn_01x04 -> Interrupt Header
- gave numbers to parts that had none: 4
Connections:
- net +5V: now also D10.2 (A), R31.1
- net GND: now also C43.2
- net SW: now also C43.1, D10.1 (K), R31.2

Commit message: Started PCB
Parts:
- removed C43: 10uF, symbol Device:C
- removed D10: DIODE, symbol pspice:DIODE
- removed R31: 10k, symbol Device:R
- added R32: R, Resistor_SMD:R_0201_0603Metric, symbol Device:R
- added R33: 10k, Resistor_SMD:R_0201_0603Metric, symbol Device:R
- C41, C42: footprint (none) -> Capacitor_SMD:CP_Elec_3x5.3
- C43: renamed from C44; footprint (none) -> Capacitor_SMD:CP_Elec_3x5.3
- J15: renamed from J3; footprint (none) -> Connector:Banana_Jack_1Pin
- R31: renamed from R30; footprint (none) -> Resistor_SMD:R_0201_0603Metric
- SW23: footprint (none) -> Button_Switch_SMD:Nidec_Copal_SH-7010A
- U34, U36: footprint (none) -> Package_DIP:DIP-20_W7.62mm
Connections:
- net +5V: now also SW23.2, R33.1
- net GND: no longer SW23.1
- net SW: now also R32.2; no longer SW23.2
- new net: R32.1, R33.2, SW23.1
Other:
- moved on the sheet: SW23
Changed lines of the file:
@@
 NoConn ~ 5450 4600
 $Comp
-L Device:R R30
+L Device:R R31
 U 1 1 61CDE2A5
 P 5450 4950
-F 0 "R30" H 5520 4996 50  0000 L CNN
+F 0 "R31" H 5520 4996 50  0000 L CNN
 F 1 "10000" H 5520 4905 50  0000 L CNN
-F 2 "" V 5380 4950 50  0001 C CNN
+F 2 "Resistor_SMD:R_0201_0603Metric" V 5380 4950 50  0001 C CNN
 F 3 "~" H 5450 4950 50  0001 C CNN
 	1    5450 4950
@@
 $EndComp
 $Comp
-L power:+5V #PWR0149
+L power:+5V #PWR0151
 U 1 1 61CDED87
 P 5450 5100
-F 0 "#PWR0149" H 5450 4950 50  0001 C CNN
+F 0 "#PWR0151" H 5450 4950 50  0001 C CNN
 F 1 "+5V" H 5465 5273 50  0000 C CNN
 F 2 "" H 5450 5100 50  0001 C CNN
@@
 $EndComp
 $Comp
-L power:+5V #PWR0145
+L power:+5V #PWR0147
 U 1 1 61CDF087
 P 4850 3200
-F 0 "#PWR0145" H 4850 3050 50  0001 C CNN
+F 0 "#PWR0147" H 4850 3050 50  0001 C CNN
 F 1 "+5V" V 4865 3328 50  0000 L CNN
 F 2 "" H 4850 3200 50  0001 C CNN
@@
 $EndComp
 $Comp
-L power:GND #PWR0146
+L power:GND #PWR0148
 U 1 1 61CDF2EC
 P 4850 5400
-F 0 "#PWR0146" H 4850 5150 50  0001 C CNN
+F 0 "#PWR0148" H 4850 5150 50  0001 C CNN
 F 1 "GND" H 4855 5227 50  0000 C CNN
 F 2 "" H 4850 5400 50  0001 C CNN
@@
 F 0 "U34" H 2600 5231 50  0000 C CNN
 F 1 "PAL16L8" H 2600 5140 50  0000 C CNN
-F 2 "" H 2600 4350 50  0001 C CNN
+F 2 "Package_DIP:DIP-20_W7.62mm" H 2600 4350 50  0001 C CNN
 F 3 "" H 2600 4350 50  0001 C CNN
 	1    2600 4350
@@
 	1750 3050 4000 3050
 $Comp
-L power:+5V #PWR0142
+L power:+5V #PWR0144
 U 1 1 61D3CF94
 P 2600 3650
-F 0 "#PWR0142" H 2600 3500 50  0001 C CNN
+F 0 "#PWR0144" H 2600 3500 50  0001 C CNN
 F 1 "+5V" V 2615 3778 50  0000 L CNN
 F 2 "" H 2600 3650 50  0001 C CNN
@@
 $EndComp
 $Comp
-L power:GND #PWR0143
+L power:GND #PWR0145
 U 1 1 61D3D228
 P 2600 4950
-F 0 "#PWR0143" H 2600 4700 50  0001 C CNN
+F 0 "#PWR0145" H 2600 4700 50  0001 C CNN
 F 1 "GND" H 2605 4777 50  0000 C CNN
 F 2 "" H 2600 4950 50  0001 C CNN
@@
 F 0 "U36" V 5754 3294 50  0000 L CNN
 F 1 "74LS244" V 5845 3294 50  0000 L CNN
-F 2 "" H 5800 2450 50  0001 C CNN
+F 2 "Package_DIP:DIP-20_W7.62mm" H 5800 2450 50  0001 C CNN
 F 3 "http://www.ti.com/lit/ds/symlink/sn74ls244.pdf" H 5800 2450 50  0001 C CNN
 	1    5800 2450
@@
 $EndComp
 $Comp
-L power:+5V #PWR0150
+L power:+5V #PWR0152
 U 1 1 61DA14DC
 P 6600 2450
-F 0 "#PWR0150" H 6600 2300 50  0001 C CNN
+F 0 "#PWR0152" H 6600 2300 50  0001 C CNN
 F 1 "+5V" H 6615 2623 50  0000 C CNN
 F 2 "" H 6600 2450 50  0001 C CNN
@@
 $EndComp
 $Comp
-L power:GND #PWR0153
+L power:GND #PWR0154
 U 1 1 61DA251B
 P 6900 2250
-F 0 "#PWR0153" H 6900 2000 50  0001 C CNN
+F 0 "#PWR0154" H 6900 2000 50  0001 C CNN
 F 1 "GND" V 6905 2122 50  0000 R CNN
 F 2 "" H 6900 2250 50  0001 C CNN
@@
 Connection ~ 6600 2450
 $Comp
-L Device:C C44
+L Device:C C43
 U 1 1 61DA5607
 P 6750 2250
-F 0 "C44" V 6498 2250 50  0000 C CNN
+F 0 "C43" V 6498 2250 50  0000 C CNN
 F 1 "0.1uF" V 6589 2250 50  0000 C CNN
-F 2 "" H 6788 2100 50  0001 C CNN
+F 2 "Capacitor_SMD:CP_Elec_3x5.3" H 6788 2100 50  0001 C CNN
 F 3 "~" H 6750 2250 50  0001 C CNN
 	1    6750 2250
@@
 $EndComp
 $Comp
-L power:GND #PWR0147
+L power:GND #PWR0149
 U 1 1 61DA801B
 P 5000 2450
-F 0 "#PWR0147" H 5000 2200 50  0001 C CNN
+F 0 "#PWR0149" H 5000 2200 50  0001 C CNN
 F 1 "GND" H 5005 2277 50  0000 C CNN
 F 2 "" H 5000 2450 50  0001 C CNN
@@
 Connection ~ 5400 1650
 $Comp
-L power:GND #PWR0148
+L power:GND #PWR0150
 U 1 1 61DABF46
 P 5400 1500
-F 0 "#PWR0148" H 5400 1250 50  0001 C CNN
+F 0 "#PWR0150" H 5400 1250 50  0001 C CNN
 F 1 "GND" H 5405 1327 50  0000 C CNN
 F 2 "" H 5400 1500 50  0001 C CNN
@@
 $EndComp
 $Comp
-L Connector_Generic:Conn_01x04 J3
+L Connector_Generic:Conn_01x04 J15
 U 1 1 61DAF565
 P 6100 1450
-F 0 "J3" V 6064 1162 50  0000 R CNN
+F 0 "J15" V 6064 1162 50  0000 R CNN
 F 1 "Interrupt Header" V 5973 1162 50  0000 R CNN
-F 2 "" H 6100 1450 50  0001 C CNN
+F 2 "Connector:Banana_Jack_1Pin" H 6100 1450 50  0001 C CNN
 F 3 "~" H 6100 1450 50  0001 C CNN
 	1    6100 1450
@@
 F 0 "C41" V 2048 3650 50  0000 C CNN
 F 1 "0.1uF" V 2139 3650 50  0000 C CNN
-F 2 "" H 2338 3500 50  0001 C CNN
+F 2 "Capacitor_SMD:CP_Elec_3x5.3" H 2338 3500 50  0001 C CNN
 F 3 "~" H 2300 3650 50  0001 C CNN
 	1    2300 3650
@@
 $EndComp
 $Comp
-L power:GND #PWR0141
+L power:GND #PWR0143
 U 1 1 61DC28AC
 P 2150 3650
-F 0 "#PWR0141" H 2150 3400 50  0001 C CNN
+F 0 "#PWR0143" H 2150 3400 50  0001 C CNN
 F 1 "GND" V 2155 3522 50  0000 R CNN
 F 2 "" H 2150 3650 50  0001 C CNN
@@
 F 0 "C42" V 4298 3200 50  0000 C CNN
 F 1 "0.1uF" V 4389 3200 50  0000 C CNN
-F 2 "" H 4588 3050 50  0001 C CNN
+F 2 "Capacitor_SMD:CP_Elec_3x5.3" H 4588 3050 50  0001 C CNN
 F 3 "~" H 4550 3200 50  0001 C CNN
 	1    4550 3200
@@
 $EndComp
 $Comp
-L power:GND #PWR0144
+L power:GND #PWR0146
 U 1 1 61DC598E
 P 4400 3200
-F 0 "#PWR0144" H 4400 2950 50  0001 C CNN
+F 0 "#PWR0146" H 4400 2950 50  0001 C CNN
 F 1 "GND" V 4405 3072 50  0000 R CNN
 F 2 "" H 4400 3200 50  0001 C CNN
@@
 	6300 2950 6300 3800
 $Comp
-L Device:R R?
-U 1 1 61BCEE13
-P 6850 3900
-AR Path="/61F6F765/61BCEE13" Ref="R?"  Part="1"
-AR Path="/61FAB268/61BCEE13" Ref="R31"  Part="1"
-F 0 "R31" H 6920 3946 50  0000 L CNN
-F 1 "10k" H 6920 3855 50  0000 L CNN
-F 2 "" V 6780 3900 50  0001 C CNN
-F 3 "~" H 6850 3900 50  0001 C CNN
-	1    6850 3900
-	-1   0    0    -1
-$EndComp
-$Comp
-L Device:C C?
-U 1 1 61BCEE19
-P 6850 4600
-AR Path="/61F6F765/61BCEE19" Ref="C?"  Part="1"
-AR Path="/61FAB268/61BCEE19" Ref="C43"  Part="1"
-F 0 "C43" H 6965 4646 50  0000 L CNN
-F 1 "10uF" H 6965 4555 50  0000 L CNN
-F 2 "" H 6888 4450 50  0001 C CNN
-F 3 "~" H 6850 4600 50  0001 C CNN
-	1    6850 4600
-	-1   0    0    -1
-$EndComp
-$Comp
-L power:GND #PWR?
-U 1 1 61BCEE1F
-P 6850 4750
-AR Path="/61F6F765/61BCEE1F" Ref="#PWR?"  Part="1"
-AR Path="/61FAB268/61BCEE1F" Ref="#PWR0152"  Part="1"
-F 0 "#PWR0152" H 6850 4500 50  0001 C CNN
-F 1 "GND" H 6855 4577 50  0000 C CNN
-F 2 "" H 6850 4750 50  0001 C CNN
-F 3 "" H 6850 4750 50  0001 C CNN
-	1    6850 4750
-	-1   0    0    -1
-$EndComp
-$Comp
 L power:+5V #PWR?
 U 1 1 61BCEE25
-P 6850 3650
+P 6850 3600
 AR Path="/61F6F765/61BCEE25" Ref="#PWR?"  Part="1"
-AR Path="/61FAB268/61BCEE25" Ref="#PWR0151"  Part="1"
-F 0 "#PWR0151" H 6850 3500 50  0001 C CNN
-F 1 "+5V" H 6865 3823 50  0000 C CNN
-F 2 "" H 6850 3650 50  0001 C CNN
-F 3 "" H 6850 3650 50  0001 C CNN
-	1    6850 3650
+AR Path="/61FAB268/61BCEE25" Ref="#PWR0153"  Part="1"
+F 0 "#PWR0153" H 6850 3450 50  0001 C CNN
+F 1 "+5V" H 6865 3773 50  0000 C CNN
+F 2 "" H 6850 3600 50  0001 C CNN
+F 3 "" H 6850 3600 50  0001 C CNN
+	1    6850 3600
 	-1   0    0    -1
 $EndComp
@@
 L Switch:SW_Push SW?
 U 1 1 61BCEE2B
-P 7500 4350
+P 6850 3900
 AR Path="/61F6F765/61BCEE2B" Ref="SW?"  Part="1"
 AR Path="/61FAB268/61BCEE2B" Ref="SW23"  Part="1"
-F 0 "SW23" H 7500 4635 50  0000 C CNN
-F 1 "SW_Push" H 7500 4544 50  0000 C CNN
-F 2 "" H 7500 4550 50  0001 C CNN
-F 3 "~" H 7500 4550 50  0001 C CNN
-	1    7500 4350
-	-1   0    0    -1
-$EndComp
-$Comp
-L power:GND #PWR?
-U 1 1 61BCEE31
-P 7700 4350
-AR Path="/61F6F765/61BCEE31" Ref="#PWR?"  Part="1"
-AR Path="/61FAB268/61BCEE31" Ref="#PWR0154"  Part="1"
-F 0 "#PWR0154" H 7700 4100 50  0001 C CNN
-F 1 "GND" H 7705 4177 50  0000 C CNN
-F 2 "" H 7700 4350 50  0001 C CNN
-F 3 "" H 7700 4350 50  0001 C CNN
-	1    7700 4350
-	-1   0    0    -1
-$EndComp
+F 0 "SW23" H 6850 4185 50  0000 C CNN
+F 1 "SW_Push" H 6850 4094 50  0000 C CNN
+F 2 "Button_Switch_SMD:Nidec_Copal_SH-7010A" H 6850 4100 50  0001 C CNN
+F 3 "~" H 6850 4100 50  0001 C CNN
+	1    6850 3900
+	0    1    -1   0
+$EndComp
+Wire Wire Line
+	6850 3600 6850 3650
+Wire Wire Line
+	6850 4350 6350 4350
+Wire Wire Line
+	6350 3850 6350 3650
+Wire Wire Line
+	6350 3650 6850 3650
+Connection ~ 6850 3650
 Wire Wire Line
 	6850 3650 6850 3700
 Wire Wire Line
-	6850 4050 6850 4350
-Wire Wire Line
-	6850 4450 6850 4350
-Connection ~ 6850 4350
-Wire Wire Line
-	7300 4350 6850 4350
-Wire Wire Line
-	6850 4350 6350 4350
-$Comp
-L pspice:DIODE D?
-U 1 1 61BCEE3D
-P 6350 4100
-AR Path="/61F6F765/61BCEE3D" Ref="D?"  Part="1"
-AR Path="/61FAB268/61BCEE3D" Ref="D10"  Part="1"
-F 0 "D10" V 6396 3972 50  0000 R CNN
-F 1 "DIODE" V 6305 3972 50  0000 R CNN
-F 2 "" H 6350 4100 50  0001 C CNN
-F 3 "~" H 6350 4100 50  0001 C CNN
-	1    6350 4100
-	0    1    -1   0
-$EndComp
-Wire Wire Line
-	6350 4350 6350 4300
+	6850 4100 6850 4350
+$Comp
+L Device:R R33
+U 1 1 61BDEED2
+P 6350 4000
+F 0 "R33" H 6420 4046 50  0000 L CNN
+F 1 "10k" H 6420 3955 50  0000 L CNN
+F 2 "Resistor_SMD:R_0201_0603Metric" V 6280 4000 50  0001 C CNN
+F 3 "~" H 6350 4000 50  0001 C CNN
+	1    6350 4000
+	1    0    0    -1
+$EndComp
+Wire Wire Line
+	6350 4150 6350 4350
+$Comp
+L Device:R R32
+U 1 1 61BE2527
+P 6000 4350
+F 0 "R32" V 5793 4350 50  0000 C CNN
+F 1 "R" V 5884 4350 50  0000 C CNN
+F 2 "Resistor_SMD:R_0201_0603Metric" V 5930 4350 50  0001 C CNN
+F 3 "~" H 6000 4350 50  0001 C CNN
+	1    6000 4350
+	0    1    1    0
+$EndComp
+Wire Wire Line
+	6150 4350 6350 4350
 Connection ~ 6350 4350
 Wire Wire Line
-	6350 4350 5850 4350
-Wire Wire Line
-	6350 3900 6350 3700
-Wire Wire Line
-	6350 3700 6850 3700
-Connection ~ 6850 3700
-Wire Wire Line
-	6850 3700 6850 3750
-Wire Wire Line
 	1750 3850 2100 3850
