File: 8279.sch (KiCad schematic (older format))
At the start: 45 parts, among them SW1 SW_Push, SW10 SW_Push, SW11 SW_Push, SW12 SW_Push, SW13 SW_Push, SW14 SW_Push, SW15 SW_Push, SW16 SW_Push, SW17 SW_Push, SW18 SW_Push, SW19 SW_Push, SW2 SW_Push, SW20 SW_Push, SW3 SW_Push, SW4 SW_Push, SW5 SW_Push, SW6 SW_Push, SW7 SW_Push, SW8 SW_Push, SW9 SW_Push, U8 74LS540, U9 74HC237

Commit message: Started PCB
Parts:
- C10: renamed from C7; footprint (none) -> Capacitor_SMD:CP_Elec_3x5.3
- C11: renamed from C8; footprint (none) -> Capacitor_SMD:CP_Elec_3x5.3
- C6: renamed from C3; footprint (none) -> Capacitor_SMD:CP_Elec_3x5.3
- C7: renamed from C4; footprint (none) -> Capacitor_SMD:CP_Elec_3x5.3
- C8: renamed from C5; footprint (none) -> Capacitor_SMD:CP_Elec_3x5.3
- C9: renamed from C6; footprint (none) -> Capacitor_SMD:CP_Elec_3x5.3
- PKDI1: footprint pkd8279 -> parts:pkd8279
- R10: renamed from R9; footprint (none) -> Resistor_SMD:R_0201_0603Metric
- R11: renamed from R10; footprint (none) -> Resistor_SMD:R_0201_0603Metric
- R2: renamed from R1; footprint (none) -> Resistor_SMD:R_0201_0603Metric
- R3: renamed from R2; footprint (none) -> Resistor_SMD:R_0201_0603Metric
- R4: renamed from R3; footprint (none) -> Resistor_SMD:R_0201_0603Metric
- R5: renamed from R4; footprint (none) -> Resistor_SMD:R_0201_0603Metric
- R6: renamed from R5; footprint (none) -> Resistor_SMD:R_0201_0603Metric
- R7: renamed from R6; footprint (none) -> Resistor_SMD:R_0201_0603Metric
- R8: renamed from R7; footprint (none) -> Resistor_SMD:R_0201_0603Metric
- R9: renamed from R8; footprint (none) -> Resistor_SMD:R_0201_0603Metric
- SW1, SW10, SW11, SW12, SW13, SW14, SW15, SW16, SW17, SW18, SW19, SW2, SW20, SW3, SW4, SW5, SW6, SW7, SW8, SW9, SWCTR1, SWINTR1, SWNMI1, SWRST1, SWSHFT1: footprint (none) -> Button_Switch_Keyboard:SW_Cherry_MX_1.00u_PCB
- U8, UPKDI1: footprint (none) -> Package_DIP:DIP-20_W7.62mm
- U9: footprint (none) -> Package_DIP:DIP-16_W10.16mm
