File: LED.sch (KiCad schematic (older format))
At the start: 20 parts

Commit message: Fixing Weirdness
Parts:
- C36, C38, C39, C40: renamed from C?; value .0000001 -> 0.1uF
- C37: renamed from C?; value C -> 0.1uF
- gave numbers to parts that had none: 15

Commit message: Started PCB
Parts:
- C36, C37, C38, C39, C40: footprint (none) -> Capacitor_SMD:CP_Elec_3x5.3
- D2, D3, D4, D5, D6, D7, D8, D9: footprint (none) -> LED_SMD:LED-APA102-2020
- RN1: footprint Resistor_THT:R_Array_SIP9 -> Resistor_SMD:R_0201_0603Metric
- U28, U29, U30, U31: footprint (none) -> Package_DIP:DIP-20_W7.62mm
Changed lines of the file:
@@
 F 0 "U29" H 5450 2731 50  0000 C CNN
 F 1 "74LS374" H 5450 2640 50  0000 C CNN
-F 2 "" H 5450 1750 50  0001 C CNN
+F 2 "Package_DIP:DIP-20_W7.62mm" H 5450 1750 50  0001 C CNN
 F 3 "http://www.ti.com/lit/gpn/sn74LS374" H 5450 1750 50  0001 C CNN
 	1    5450 1750
@@
 F 0 "U30" H 5450 4831 50  0000 C CNN
 F 1 "74LS374" H 5450 4740 50  0000 C CNN
-F 2 "" H 5450 3850 50  0001 C CNN
+F 2 "Package_DIP:DIP-20_W7.62mm" H 5450 3850 50  0001 C CNN
 F 3 "http://www.ti.com/lit/gpn/sn74LS374" H 5450 3850 50  0001 C CNN
 	1    5450 3850
@@
 $EndComp
 $Comp
-L power:+5V #PWR0135
+L power:+5V #PWR0137
 U 1 1 61F8AC15
 P 6650 1850
-F 0 "#PWR0135" H 6650 1700 50  0001 C CNN
+F 0 "#PWR0137" H 6650 1700 50  0001 C CNN
 F 1 "+5V" V 6665 1978 50  0000 L CNN
 F 2 "" H 6650 1850 50  0001 C CNN
@@
 $EndComp
 $Comp
-L power:+5V #PWR0136
+L power:+5V #PWR0138
 U 1 1 61F8BABB
 P 6650 1950
-F 0 "#PWR0136" H 6650 1800 50  0001 C CNN
+F 0 "#PWR0138" H 6650 1800 50  0001 C CNN
 F 1 "+5V" V 6665 2078 50  0000 L CNN
 F 2 "" H 6650 1950 50  0001 C CNN
@@
 $EndComp
 $Comp
-L power:+5V #PWR0137
+L power:+5V #PWR0139
 U 1 1 61F8BDF1
 P 6650 3950
-F 0 "#PWR0137" H 6650 3800 50  0001 C CNN
+F 0 "#PWR0139" H 6650 3800 50  0001 C CNN
 F 1 "+5V" V 6665 4078 50  0000 L CNN
 F 2 "" H 6650 3950 50  0001 C CNN
@@
 $EndComp
 $Comp
-L power:+5V #PWR0138
+L power:+5V #PWR0140
 U 1 1 61F8C723
 P 6650 4050
-F 0 "#PWR0138" H 6650 3900 50  0001 C CNN
+F 0 "#PWR0140" H 6650 3900 50  0001 C CNN
 F 1 "+5V" V 6665 4178 50  0000 L CNN
 F 2 "" H 6650 4050 50  0001 C CNN
@@
 F 0 "U28" H 3050 4731 50  0000 C CNN
 F 1 "PAL16L8" H 3050 4640 50  0000 C CNN
-F 2 "" H 3050 3850 50  0001 C CNN
+F 2 "Package_DIP:DIP-20_W7.62mm" H 3050 3850 50  0001 C CNN
 F 3 "" H 3050 3850 50  0001 C CNN
 	1    3050 3850
@@
 F 0 "U31" H 5450 6731 50  0000 C CNN
 F 1 "74LS374" H 5450 6640 50  0000 C CNN
-F 2 "" H 5450 5750 50  0001 C CNN
+F 2 "Package_DIP:DIP-20_W7.62mm" H 5450 5750 50  0001 C CNN
 F 3 "http://www.ti.com/lit/gpn/sn74LS374" H 5450 5750 50  0001 C CNN
 	1    5450 5750
@@
 	4650 6150 4950 6150
 $Comp
-L power:GND #PWR094
+L power:GND #PWR0127
 U 1 1 61F9FAC6
 P 4950 6250
-F 0 "#PWR094" H 4950 6000 50  0001 C CNN
+F 0 "#PWR0127" H 4950 6000 50  0001 C CNN
 F 1 "GND" H 4955 6077 50  0000 C CNN
 F 2 "" H 4950 6250 50  0001 C CNN
@@
 $EndComp
 $Comp
-L power:GND #PWR0134
+L power:GND #PWR0136
 U 1 1 61F9FBDA
 P 5450 6550
-F 0 "#PWR0134" H 5450 6300 50  0001 C CNN
+F 0 "#PWR0136" H 5450 6300 50  0001 C CNN
 F 1 "GND" H 5455 6377 50  0000 C CNN
 F 2 "" H 5450 6550 50  0001 C CNN
@@
 A[9]
 $Comp
-L power:GND #PWR0132
+L power:GND #PWR0134
 U 1 1 61FD462E
 P 5450 4650
-F 0 "#PWR0132" H 5450 4400 50  0001 C CNN
+F 0 "#PWR0134" H 5450 4400 50  0001 C CNN
 F 1 "GND" V 5455 4522 50  0000 R CNN
 F 2 "" H 5450 4650 50  0001 C CNN
@@
 $EndComp
 $Comp
-L power:GND #PWR099
+L power:GND #PWR0132
 U 1 1 61FD8EE8
 P 5450 2550
-F 0 "#PWR099" H 5450 2300 50  0001 C CNN
+F 0 "#PWR0132" H 5450 2300 50  0001 C CNN
 F 1 "GND" H 5455 2377 50  0000 C CNN
 F 2 "" H 5450 2550 50  0001 C CNN
@@
 $EndComp
 $Comp
-L power:+5V #PWR0133
+L power:+5V #PWR0135
 U 1 1 61FD91E3
 P 5450 4950
-F 0 "#PWR0133" H 5450 4800 50  0001 C CNN
+F 0 "#PWR0135" H 5450 4800 50  0001 C CNN
 F 1 "+5V" V 5465 5078 50  0000 L CNN
 F 2 "" H 5450 4950 50  0001 C CNN
@@
 F 0 "C39" V 4898 4950 50  0000 C CNN
 F 1 "0.1uF" V 4989 4950 50  0000 C CNN
-F 2 "" H 5188 4800 50  0001 C CNN
+F 2 "Capacitor_SMD:CP_Elec_3x5.3" H 5188 4800 50  0001 C CNN
 F 3 "~" H 5150 4950 50  0001 C CNN
 	1    5150 4950
@@
 $EndComp
 $Comp
-L power:GND #PWR097
+L power:GND #PWR0130
 U 1 1 61FDBC67
 P 5000 4950
-F 0 "#PWR097" H 5000 4700 50  0001 C CNN
+F 0 "#PWR0130" H 5000 4700 50  0001 C CNN
 F 1 "GND" H 5005 4777 50  0000 C CNN
 F 2 "" H 5000 4950 50  0001 C CNN
@@
 $EndComp
 $Comp
-L power:+5V #PWR0100
+L power:+5V #PWR0133
 U 1 1 61FDBFBE
 P 5450 3050
-F 0 "#PWR0100" H 5450 2900 50  0001 C CNN
+F 0 "#PWR0133" H 5450 2900 50  0001 C CNN
 F 1 "+5V" V 5465 3178 50  0000 L CNN
 F 2 "" H 5450 3050 50  0001 C CNN
@@
 F 0 "C38" V 4898 3050 50  0000 C CNN
 F 1 "0.1uF" V 4989 3050 50  0000 C CNN
-F 2 "" H 5188 2900 50  0001 C CNN
+F 2 "Capacitor_SMD:CP_Elec_3x5.3" H 5188 2900 50  0001 C CNN
 F 3 "~" H 5150 3050 50  0001 C CNN
 	1    5150 3050
@@
 $EndComp
 $Comp
-L power:GND #PWR096
+L power:GND #PWR0129
 U 1 1 61FE4A7C
 P 5000 3050
-F 0 "#PWR096" H 5000 2800 50  0001 C CNN
+F 0 "#PWR0129" H 5000 2800 50  0001 C CNN
 F 1 "GND" H 5005 2877 50  0000 C CNN
 F 2 "" H 5000 3050 50  0001 C CNN
@@
 $EndComp
 $Comp
-L power:GND #PWR093
+L power:GND #PWR0126
 U 1 1 61FE4DA9
 P 3050 4450
-F 0 "#PWR093" H 3050 4200 50  0001 C CNN
+F 0 "#PWR0126" H 3050 4200 50  0001 C CNN
 F 1 "GND" H 3055 4277 50  0000 C CNN
 F 2 "" H 3050 4450 50  0001 C CNN
@@
 $EndComp
 $Comp
-L power:+5V #PWR092
+L power:+5V #PWR0125
 U 1 1 61FE4EE5
 P 3050 3150
-F 0 "#PWR092" H 3050 3000 50  0001 C CNN
+F 0 "#PWR0125" H 3050 3000 50  0001 C CNN
 F 1 "+5V" V 3065 3278 50  0000 L CNN
 F 2 "" H 3050 3150 50  0001 C CNN
@@
 $EndComp
 $Comp
-L power:+5V #PWR098
+L power:+5V #PWR0131
 U 1 1 61FE6201
 P 5450 950
-F 0 "#PWR098" H 5450 800 50  0001 C CNN
+F 0 "#PWR0131" H 5450 800 50  0001 C CNN
 F 1 "+5V" V 5465 1078 50  0000 L CNN
 F 2 "" H 5450 950 50  0001 C CNN
@@
 F 0 "C36" V 2498 3150 50  0000 C CNN
 F 1 "0.1uF" V 2589 3150 50  0000 C CNN
-F 2 "" H 2788 3000 50  0001 C CNN
+F 2 "Capacitor_SMD:CP_Elec_3x5.3" H 2788 3000 50  0001 C CNN
 F 3 "~" H 2750 3150 50  0001 C CNN
 	1    2750 3150
@@
 F 0 "C37" V 4898 950 50  0000 C CNN
 F 1 "0.1uF" V 4989 950 50  0000 C CNN
-F 2 "" H 5188 800 50  0001 C CNN
+F 2 "Capacitor_SMD:CP_Elec_3x5.3" H 5188 800 50  0001 C CNN
 F 3 "~" H 5150 950 50  0001 C CNN
 	1    5150 950
@@
 Connection ~ 3050 3150
 $Comp
-L power:GND #PWR091
+L power:GND #PWR0124
 U 1 1 61FEBB63
 P 2600 3150
-F 0 "#PWR091" H 2600 2900 50  0001 C CNN
+F 0 "#PWR0124" H 2600 2900 50  0001 C CNN
 F 1 "GND" V 2605 3022 50  0000 R CNN
 F 2 "" H 2600 3150 50  0001 C CNN
@@
 $EndComp
 $Comp
-L power:GND #PWR095
+L power:GND #PWR0128
 U 1 1 61FEBC68
 P 5000 950
-F 0 "#PWR095" H 5000 700 50  0001 C CNN
+F 0 "#PWR0128" H 5000 700 50  0001 C CNN
 F 1 "GND" V 5005 822 50  0000 R CNN
 F 2 "" H 5000 950 50  0001 C CNN
@@
 F 0 "D2" V 7389 4182 50  0000 R CNN
 F 1 "LED" V 7298 4182 50  0000 R CNN
-F 2 "" H 7350 4300 50  0001 C CNN
+F 2 "LED_SMD:LED-APA102-2020" H 7350 4300 50  0001 C CNN
 F 3 "~" H 7350 4300 50  0001 C CNN
 	1    7350 4300
@@
 F 0 "D3" V 7739 4182 50  0000 R CNN
 F 1 "LED" V 7648 4182 50  0000 R CNN
-F 2 "" H 7700 4300 50  0001 C CNN
+F 2 "LED_SMD:LED-APA102-2020" H 7700 4300 50  0001 C CNN
 F 3 "~" H 7700 4300 50  0001 C CNN
 	1    7700 4300
@@
 F 0 "D4" V 8089 4182 50  0000 R CNN
 F 1 "LED" V 7998 4182 50  0000 R CNN
-F 2 "" H 8050 4300 50  0001 C CNN
+F 2 "LED_SMD:LED-APA102-2020" H 8050 4300 50  0001 C CNN
 F 3 "~" H 8050 4300 50  0001 C CNN
 	1    8050 4300
@@
 F 0 "D5" V 8439 4182 50  0000 R CNN
 F 1 "LED" V 8348 4182 50  0000 R CNN
-F 2 "" H 8400 4300 50  0001 C CNN
+F 2 "LED_SMD:LED-APA102-2020" H 8400 4300 50  0001 C CNN
 F 3 "~" H 8400 4300 50  0001 C CNN
 	1    8400 4300
@@
 F 0 "D6" V 8789 4182 50  0000 R CNN
 F 1 "LED" V 8698 4182 50  0000 R CNN
-F 2 "" H 8750 4300 50  0001 C CNN
+F 2 "LED_SMD:LED-APA102-2020" H 8750 4300 50  0001 C CNN
 F 3 "~" H 8750 4300 50  0001 C CNN
 	1    8750 4300
@@
 F 0 "D7" V 9139 4182 50  0000 R CNN
 F 1 "LED" V 9048 4182 50  0000 R CNN
-F 2 "" H 9100 4300 50  0001 C CNN
+F 2 "LED_SMD:LED-APA102-2020" H 9100 4300 50  0001 C CNN
 F 3 "~" H 9100 4300 50  0001 C CNN
 	1    9100 4300
@@
 F 0 "D8" V 9489 4182 50  0000 R CNN
 F 1 "LED" V 9398 4182 50  0000 R CNN
-F 2 "" H 9450 4300 50  0001 C CNN
+F 2 "LED_SMD:LED-APA102-2020" H 9450 4300 50  0001 C CNN
 F 3 "~" H 9450 4300 50  0001 C CNN
 	1    9450 4300
@@
 F 0 "D9" V 9789 4182 50  0000 R CNN
 F 1 "LED" V 9698 4182 50  0000 R CNN
-F 2 "" H 9750 4300 50  0001 C CNN
+F 2 "LED_SMD:LED-APA102-2020" H 9750 4300 50  0001 C CNN
 F 3 "~" H 9750 4300 50  0001 C CNN
 	1    9750 4300
@@
 F 0 "RN1" H 7570 3096 50  0000 R CNN
 F 1 "R_Network08" H 7570 3005 50  0000 R CNN
-F 2 "Resistor_THT:R_Array_SIP9" V 8525 3050 50  0001 C CNN
+F 2 "Resistor_SMD:R_0201_0603Metric" V 8525 3050 50  0001 C CNN
 F 3 "http://www.vishay.com/docs/31509/csc.pdf" H 8050 3050 50  0001 C CNN
 	1    8050 3050
@@
 F 0 "C40" V 7848 2100 50  0000 C CNN
 F 1 "0.1uF" V 7939 2100 50  0000 C CNN
-F 2 "" H 8138 1950 50  0001 C CNN
+F 2 "Capacitor_SMD:CP_Elec_3x5.3" H 8138 1950 50  0001 C CNN
 F 3 "~" H 8100 2100 50  0001 C CNN
 	1    8100 2100
@@
 $EndComp
 $Comp
-L power:GND #PWR0139
+L power:GND #PWR0141
 U 1 1 620543DA
 P 7950 2100
-F 0 "#PWR0139" H 7950 1850 50  0001 C CNN
+F 0 "#PWR0141" H 7950 1850 50  0001 C CNN
 F 1 "GND" V 7955 1972 50  0000 R CNN
 F 2 "" H 7950 2100 50  0001 C CNN
@@
 	8450 2500 8450 2850
 $Comp
-L power:+5V #PWR0140
+L power:+5V #PWR0142
 U 1 1 620582F3
 P 8750 2500
-F 0 "#PWR0140" H 8750 2350 50  0001 C CNN
+F 0 "#PWR0142" H 8750 2350 50  0001 C CNN
 F 1 "+5V" V 8765 2628 50  0000 L CNN
 F 2 "" H 8750 2500 50  0001 C CNN
