File: SRAM.sch (KiCad schematic (older format))
At the start: 9 parts, among them U13 PAL16L8, U14 CY7C199, U15 CY7C199, U16 CY7C199, U17 CY7C199

Commit message: Started PCB
Parts:
- C14: renamed from C11; footprint (none) -> Capacitor_SMD:CP_Elec_3x5.3
- C15: renamed from C12; footprint (none) -> Capacitor_SMD:CP_Elec_3x5.3
- C16: renamed from C13; footprint (none) -> Capacitor_SMD:CP_Elec_3x5.3
- C17: renamed from C14; footprint (none) -> Capacitor_SMD:CP_Elec_3x5.3
- U13: footprint (none) -> Package_DIP:DIP-20_W7.62mm
- U14, U15, U16, U17: footprint (none) -> Package_DIP:DIP-28_W7.62mm
Changed lines of the file:
@@
 F 0 "U14" H 3900 3350 50  0000 C CNN
 F 1 "CY7C199" H 3900 3250 50  0000 C CNN
-F 2 "" H 3900 2600 50  0001 C CNN
+F 2 "Package_DIP:DIP-28_W7.62mm" H 3900 2600 50  0001 C CNN
 F 3 "" H 3900 2600 50  0001 C CNN
 	1    3900 2600
@@
 	1300 1400 1200 1400
 $Comp
-L power:GND #PWR074
+L power:GND #PWR079
 U 1 1 61D25220
 P 3900 3800
-F 0 "#PWR074" H 3900 3550 50  0001 C CNN
+F 0 "#PWR079" H 3900 3550 50  0001 C CNN
 F 1 "GND" H 3905 3627 50  0000 C CNN
 F 2 "" H 3900 3800 50  0001 C CNN
@@
 $EndComp
 $Comp
-L power:+5V #PWR073
+L power:+5V #PWR078
 U 1 1 61D254C1
 P 3900 1400
-F 0 "#PWR073" H 3900 1250 50  0001 C CNN
+F 0 "#PWR078" H 3900 1250 50  0001 C CNN
 F 1 "+5V" V 3915 1528 50  0000 L CNN
 F 2 "" H 3900 1400 50  0001 C CNN
@@
 $EndComp
 $Comp
-L power:+5V #PWR069
+L power:+5V #PWR074
 U 1 1 61D260A2
 P 2200 3600
-F 0 "#PWR069" H 2200 3450 50  0001 C CNN
+F 0 "#PWR074" H 2200 3450 50  0001 C CNN
 F 1 "+5V" V 2215 3728 50  0000 L CNN
 F 2 "" H 2200 3600 50  0001 C CNN
@@
 $EndComp
 $Comp
-L power:GND #PWR070
+L power:GND #PWR075
 U 1 1 61D263BA
 P 2200 4900
-F 0 "#PWR070" H 2200 4650 50  0001 C CNN
+F 0 "#PWR075" H 2200 4650 50  0001 C CNN
 F 1 "GND" H 2205 4727 50  0000 C CNN
 F 2 "" H 2200 4900 50  0001 C CNN
@@
 F 0 "U15" H 3900 6350 50  0000 C CNN
 F 1 "CY7C199" H 3900 6250 50  0000 C CNN
-F 2 "" H 3900 5600 50  0001 C CNN
+F 2 "Package_DIP:DIP-28_W7.62mm" H 3900 5600 50  0001 C CNN
 F 3 "" H 3900 5600 50  0001 C CNN
 	1    3900 5600
@@
 	3000 6500 3300 6500
 $Comp
-L power:GND #PWR076
+L power:GND #PWR081
 U 1 1 61D930C9
 P 3900 6800
-F 0 "#PWR076" H 3900 6550 50  0001 C CNN
+F 0 "#PWR081" H 3900 6550 50  0001 C CNN
 F 1 "GND" H 3905 6627 50  0000 C CNN
 F 2 "" H 3900 6800 50  0001 C CNN
@@
 $EndComp
 $Comp
-L power:+5V #PWR075
+L power:+5V #PWR080
 U 1 1 61D930D3
 P 3900 4400
-F 0 "#PWR075" H 3900 4250 50  0001 C CNN
+F 0 "#PWR080" H 3900 4250 50  0001 C CNN
 F 1 "+5V" V 3915 4528 50  0000 L CNN
 F 2 "" H 3900 4400 50  0001 C CNN
@@
 	4900 6300 5500 6300
 $Comp
-L power:GND #PWR082
+L power:GND #PWR087
 U 1 1 61DCF52C
 P 6100 6800
-F 0 "#PWR082" H 6100 6550 50  0001 C CNN
+F 0 "#PWR087" H 6100 6550 50  0001 C CNN
 F 1 "GND" H 6105 6627 50  0000 C CNN
 F 2 "" H 6100 6800 50  0001 C CNN
@@
 $EndComp
 $Comp
-L power:+5V #PWR081
+L power:+5V #PWR086
 U 1 1 61DCF532
 P 6100 4400
-F 0 "#PWR081" H 6100 4250 50  0001 C CNN
+F 0 "#PWR086" H 6100 4250 50  0001 C CNN
 F 1 "+5V" V 6115 4528 50  0000 L CNN
 F 2 "" H 6100 4400 50  0001 C CNN
@@
 F 0 "U16" H 6100 3400 50  0000 C CNN
 F 1 "CY7C199" H 6100 3300 50  0000 C CNN
-F 2 "" H 6100 2600 50  0001 C CNN
+F 2 "Package_DIP:DIP-28_W7.62mm" H 6100 2600 50  0001 C CNN
 F 3 "" H 6100 2600 50  0001 C CNN
 	1    6100 2600
@@
 	4900 3300 5500 3300
 $Comp
-L power:GND #PWR080
+L power:GND #PWR085
 U 1 1 61DD75EF
 P 6100 3800
-F 0 "#PWR080" H 6100 3550 50  0001 C CNN
+F 0 "#PWR085" H 6100 3550 50  0001 C CNN
 F 1 "GND" H 6105 3627 50  0000 C CNN
 F 2 "" H 6100 3800 50  0001 C CNN
@@
 $EndComp
 $Comp
-L power:+5V #PWR079
+L power:+5V #PWR084
 U 1 1 61DD75F5
 P 6100 1400
-F 0 "#PWR079" H 6100 1250 50  0001 C CNN
+F 0 "#PWR084" H 6100 1250 50  0001 C CNN
 F 1 "+5V" V 6115 1528 50  0000 L CNN
 F 2 "" H 6100 1400 50  0001 C CNN
@@
 F 0 "U13" H 2200 5181 50  0000 C CNN
 F 1 "PAL16L8" H 2200 5090 50  0000 C CNN
-F 2 "" H 2200 4300 50  0001 C CNN
+F 2 "Package_DIP:DIP-20_W7.62mm" H 2200 4300 50  0001 C CNN
 F 3 "" H 2200 4300 50  0001 C CNN
 	1    2200 4300
@@
 NoConn ~ 1700 4500
 $Comp
-L power:GND #PWR072
+L power:GND #PWR077
 U 1 1 61B7788D
 P 3700 4400
-F 0 "#PWR072" H 3700 4150 50  0001 C CNN
+F 0 "#PWR077" H 3700 4150 50  0001 C CNN
 F 1 "GND" V 3705 4272 50  0000 R CNN
 F 2 "" H 3700 4400 50  0001 C CNN
@@
 $EndComp
 $Comp
-L Device:C_Small C12
+L Device:C_Small C15
 U 1 1 61B929A4
 P 3800 4400
-F 0 "C12" V 3571 4400 50  0000 C CNN
+F 0 "C15" V 3571 4400 50  0000 C CNN
 F 1 "0.1uF" V 3662 4400 50  0000 C CNN
-F 2 "" H 3800 4400 50  0001 C CNN
+F 2 "Capacitor_SMD:CP_Elec_3x5.3" H 3800 4400 50  0001 C CNN
 F 3 "~" H 3800 4400 50  0001 C CNN
 	1    3800 4400
@@
 F 0 "U17" H 6100 6250 50  0000 C CNN
 F 1 "CY7C199" H 6100 6150 50  0000 C CNN
-F 2 "" H 6100 5600 50  0001 C CNN
+F 2 "Package_DIP:DIP-28_W7.62mm" H 6100 5600 50  0001 C CNN
 F 3 "" H 6100 5600 50  0001 C CNN
 	1    6100 5600
@@
 $EndComp
 $Comp
-L Device:C_Small C14
+L Device:C_Small C17
 U 1 1 61BAF1F0
 P 6000 4400
-F 0 "C14" V 5771 4400 50  0000 C CNN
+F 0 "C17" V 5771 4400 50  0000 C CNN
 F 1 "0.1uF" V 5862 4400 50  0000 C CNN
-F 2 "" H 6000 4400 50  0001 C CNN
+F 2 "Capacitor_SMD:CP_Elec_3x5.3" H 6000 4400 50  0001 C CNN
 F 3 "~" H 6000 4400 50  0001 C CNN
 	1    6000 4400
@@
 Connection ~ 6100 4400
 $Comp
-L power:GND #PWR078
+L power:GND #PWR083
 U 1 1 61BAFEEF
 P 5900 4400
-F 0 "#PWR078" H 5900 4150 50  0001 C CNN
+F 0 "#PWR083" H 5900 4150 50  0001 C CNN
 F 1 "GND" V 5905 4272 50  0000 R CNN
 F 2 "" H 5900 4400 50  0001 C CNN
@@
 $EndComp
 $Comp
-L Device:C_Small C13
+L Device:C_Small C16
 U 1 1 61BB084F
 P 6000 1400
-F 0 "C13" V 5771 1400 50  0000 C CNN
+F 0 "C16" V 5771 1400 50  0000 C CNN
 F 1 "0.1uF" V 5862 1400 50  0000 C CNN
-F 2 "" H 6000 1400 50  0001 C CNN
+F 2 "Capacitor_SMD:CP_Elec_3x5.3" H 6000 1400 50  0001 C CNN
 F 3 "~" H 6000 1400 50  0001 C CNN
 	1    6000 1400
@@
 Connection ~ 6100 1400
 $Comp
-L Device:C_Small C11
+L Device:C_Small C14
 U 1 1 61BB16C0
 P 3800 1400
-F 0 "C11" V 3571 1400 50  0000 C CNN
+F 0 "C14" V 3571 1400 50  0000 C CNN
 F 1 "0.1uF" V 3662 1400 50  0000 C CNN
-F 2 "" H 3800 1400 50  0001 C CNN
+F 2 "Capacitor_SMD:CP_Elec_3x5.3" H 3800 1400 50  0001 C CNN
 F 3 "~" H 3800 1400 50  0001 C CNN
 	1    3800 1400
@@
 Connection ~ 3900 1400
 $Comp
-L power:GND #PWR071
+L power:GND #PWR076
 U 1 1 61BB1D2E
 P 3700 1400
-F 0 "#PWR071" H 3700 1150 50  0001 C CNN
+F 0 "#PWR076" H 3700 1150 50  0001 C CNN
 F 1 "GND" V 3705 1272 50  0000 R CNN
 F 2 "" H 3700 1400 50  0001 C CNN
@@
 $EndComp
 $Comp
-L power:GND #PWR077
+L power:GND #PWR082
 U 1 1 61BB20A9
 P 5900 1400
-F 0 "#PWR077" H 5900 1150 50  0001 C CNN
+F 0 "#PWR082" H 5900 1150 50  0001 C CNN
 F 1 "GND" V 5905 1272 50  0000 R CNN
 F 2 "" H 5900 1400 50  0001 C CNN
