File: UART.sch (KiCad schematic (older format))
At the start: 7 parts, among them J2 DSUB-9, U10 PAL16L8, U11 16550, U12 max235cpg

Commit message: Started PCB
Parts:
- C12: renamed from C9; footprint (none) -> Capacitor_SMD:CP_Elec_3x5.3
- C13: renamed from C10; footprint (none) -> Capacitor_SMD:CP_Elec_3x5.3
- J14: renamed from J2; footprint DSUB-9 -> parts:DSUB-9
- R12: renamed from R11; footprint (none) -> Resistor_SMD:R_0201_0603Metric
- U10: footprint (none) -> Package_DIP:DIP-20_W7.62mm
- U12: footprint max235cpg -> Package_DIP:DIP-24_W15.24mm
Changed lines of the file:
@@
 $EndDescr
 $Comp
-L DSUB-9:DSUB-9 J2
+L DSUB-9:DSUB-9 J14
 U 1 1 6249A35C
 P 9500 2150
-F 0 "J2" V 9839 2278 60  0000 L CNN
+F 0 "J14" V 9839 2278 60  0000 L CNN
 F 1 "DSUB-9" V 9945 2278 60  0000 L CNN
-F 2 "DSUB-9" H 10100 1790 60  0001 C CNN
+F 2 "parts:DSUB-9" H 10100 1790 60  0001 C CNN
 F 3 "" H 9500 2150 60  0000 C CNN
 	1    9500 2150
@@
 $EndComp
 $Comp
-L power:GND #PWR059
+L power:GND #PWR064
 U 1 1 6249AAEF
 P 4200 3800
-F 0 "#PWR059" H 4200 3550 50  0001 C CNN
+F 0 "#PWR064" H 4200 3550 50  0001 C CNN
 F 1 "GND" V 4205 3672 50  0000 R CNN
 F 2 "" H 4200 3800 50  0001 C CNN
@@
 $EndComp
 $Comp
-L power:GND #PWR060
+L power:GND #PWR065
 U 1 1 6249B12C
 P 4200 3900
-F 0 "#PWR060" H 4200 3650 50  0001 C CNN
+F 0 "#PWR065" H 4200 3650 50  0001 C CNN
 F 1 "GND" V 4205 3772 50  0000 R CNN
 F 2 "" H 4200 3900 50  0001 C CNN
@@
 $EndComp
 $Comp
-L power:GND #PWR064
+L power:GND #PWR069
 U 1 1 6249B47B
 P 5200 4600
-F 0 "#PWR064" H 5200 4350 50  0001 C CNN
+F 0 "#PWR069" H 5200 4350 50  0001 C CNN
 F 1 "GND" H 5205 4427 50  0000 C CNN
 F 2 "" H 5200 4600 50  0001 C CNN
@@
 $EndComp
 $Comp
-L power:GND #PWR061
+L power:GND #PWR066
 U 1 1 6249C757
 P 4200 4100
-F 0 "#PWR061" H 4200 3850 50  0001 C CNN
+F 0 "#PWR066" H 4200 3850 50  0001 C CNN
 F 1 "GND" V 4205 3972 50  0000 R CNN
 F 2 "" H 4200 4100 50  0001 C CNN
@@
 	4200 2700 4200 2800
 $Comp
-L Device:R R11
+L Device:R R12
 U 1 1 624A138D
 P 4050 2800
-F 0 "R11" V 4050 2800 50  0000 C CNN
+F 0 "R12" V 4050 2800 50  0000 C CNN
 F 1 "R" V 3934 2800 50  0000 C CNN
-F 2 "" V 3980 2800 50  0001 C CNN
+F 2 "Resistor_SMD:R_0201_0603Metric" V 3980 2800 50  0001 C CNN
 F 3 "~" H 4050 2800 50  0001 C CNN
 	1    4050 2800
@@
 F 0 "U10" H 3000 3581 50  0000 C CNN
 F 1 "PAL16L8" H 3000 3490 50  0000 C CNN
-F 2 "" H 3000 2700 50  0001 C CNN
+F 2 "Package_DIP:DIP-20_W7.62mm" H 3000 2700 50  0001 C CNN
 F 3 "" H 3000 2700 50  0001 C CNN
 	1    3000 2700
@@
 	1750 4300 1750 1900
 $Comp
-L power:GND #PWR068
+L power:GND #PWR073
 U 1 1 624C8D96
 P 9500 2550
-F 0 "#PWR068" H 9500 2300 50  0001 C CNN
+F 0 "#PWR073" H 9500 2300 50  0001 C CNN
 F 1 "GND" H 9505 2377 50  0000 C CNN
 F 2 "" H 9500 2550 50  0001 C CNN
@@
 F 0 "U12" H 9850 1787 60  0000 C CNN
 F 1 "max235cpg" H 9850 1681 60  0000 C CNN
-F 2 "max235cpg" H 9850 1640 60  0001 C CNN
+F 2 "Package_DIP:DIP-24_W15.24mm" H 9850 1640 60  0001 C CNN
 F 3 "" H 8550 1400 60  0000 C CNN
 	1    8550 1400
@@
 NoConn ~ 8350 4000
 $Comp
-L power:GND #PWR058
+L power:GND #PWR062
 U 1 1 6255AC9F
 P 3000 3300
-F 0 "#PWR058" H 3000 3050 50  0001 C CNN
+F 0 "#PWR062" H 3000 3050 50  0001 C CNN
 F 1 "GND" H 3005 3127 50  0000 C CNN
 F 2 "" H 3000 3300 50  0001 C CNN
@@
 Connection ~ 8250 4000
 $Comp
-L power:GND #PWR067
+L power:GND #PWR072
 U 1 1 6255481D
 P 8250 4000
-F 0 "#PWR067" H 8250 3750 50  0001 C CNN
+F 0 "#PWR072" H 8250 3750 50  0001 C CNN
 F 1 "GND" H 8255 3827 50  0000 C CNN
 F 2 "" H 8250 4000 50  0001 C CNN
@@
 Reset
 $Comp
-L power:+5V #PWR057
+L power:+5V #PWR061
 U 1 1 62583790
 P 3000 2000
-F 0 "#PWR057" H 3000 1850 50  0001 C CNN
+F 0 "#PWR061" H 3000 1850 50  0001 C CNN
 F 1 "+5V" V 3015 2128 50  0000 L CNN
 F 2 "" H 3000 2000 50  0001 C CNN
@@
 $EndComp
 $Comp
-L power:+5V #PWR063
+L power:+5V #PWR068
 U 1 1 62586C4F
 P 5200 1200
-F 0 "#PWR063" H 5200 1050 50  0001 C CNN
+F 0 "#PWR068" H 5200 1050 50  0001 C CNN
 F 1 "+5V" V 5215 1328 50  0000 L CNN
 F 2 "" H 5200 1200 50  0001 C CNN
@@
 P 5000 1200
 AR Path="/62BD3577/61C0C203" Ref="#PWR?"  Part="1"
-AR Path="/6241A5BB/61C0C203" Ref="#PWR062"  Part="1"
-F 0 "#PWR062" H 5000 950 50  0001 C CNN
+AR Path="/6241A5BB/61C0C203" Ref="#PWR067"  Part="1"
+F 0 "#PWR067" H 5000 950 50  0001 C CNN
 F 1 "GND" H 5005 1027 50  0000 C CNN
 F 2 "" H 5000 1200 50  0001 C CNN
@@
 P 5100 1200
 AR Path="/62BD3577/61C0C209" Ref="C?"  Part="1"
-AR Path="/6241A5BB/61C0C209" Ref="C9"  Part="1"
-F 0 "C9" H 5192 1246 50  0000 L CNN
+AR Path="/6241A5BB/61C0C209" Ref="C12"  Part="1"
+F 0 "C12" H 5192 1246 50  0000 L CNN
 F 1 "0.1uF" H 5192 1155 50  0000 L CNN
-F 2 "" H 5100 1200 50  0001 C CNN
+F 2 "Capacitor_SMD:CP_Elec_3x5.3" H 5100 1200 50  0001 C CNN
 F 3 "~" H 5100 1200 50  0001 C CNN
 	1    5100 1200
@@
 P 7450 1300
 AR Path="/62BD3577/61C106FC" Ref="C?"  Part="1"
-AR Path="/6241A5BB/61C106FC" Ref="C10"  Part="1"
-F 0 "C10" H 7542 1346 50  0000 L CNN
+AR Path="/6241A5BB/61C106FC" Ref="C13"  Part="1"
+F 0 "C13" H 7542 1346 50  0000 L CNN
 F 1 "0.1uF" H 7542 1255 50  0000 L CNN
-F 2 "" H 7450 1300 50  0001 C CNN
+F 2 "Capacitor_SMD:CP_Elec_3x5.3" H 7450 1300 50  0001 C CNN
 F 3 "~" H 7450 1300 50  0001 C CNN
 	1    7450 1300
@@
 Connection ~ 7550 1300
 $Comp
-L power:GND #PWR066
+L power:GND #PWR071
 U 1 1 61C1802F
 P 7550 1300
-F 0 "#PWR066" H 7550 1050 50  0001 C CNN
+F 0 "#PWR071" H 7550 1050 50  0001 C CNN
 F 1 "GND" H 7500 1100 50  0000 C CNN
 F 2 "" H 7550 1300 50  0001 C CNN
@@
 $EndComp
 $Comp
-L power:+5V #PWR065
+L power:+5V #PWR070
 U 1 1 61C2C387
 P 7350 1300
-F 0 "#PWR065" H 7350 1150 50  0001 C CNN
+F 0 "#PWR070" H 7350 1150 50  0001 C CNN
 F 1 "+5V" V 7450 1350 50  0000 L CNN
 F 2 "" H 7350 1300 50  0001 C CNN
@@
 Text HLabel 1650 2000 0    50   Input ~ 0
 Clk
-Wire Bus Line
-	3900 2300 3900 2500
-Wire Bus Line
-	3700 2300 3700 2600
-Wire Bus Line
-	2250 1400 2250 2900
-Wire Bus Line
-	3900 1300 3900 2100
-$Comp
-L power:+5V #PWR07
+$Comp
+L power:+5V #PWR063
 U 1 1 61FC357D
 P 3900 2800
-F 0 "#PWR07" H 3900 2650 50  0001 C CNN
+F 0 "#PWR063" H 3900 2650 50  0001 C CNN
 F 1 "+5V" V 3915 2928 50  0000 L CNN
 F 2 "" H 3900 2800 50  0001 C CNN
@@
 	0    -1   -1   0
 $EndComp
+Wire Bus Line
+	3900 2300 3900 2500
+Wire Bus Line
+	3700 2300 3700 2600
+Wire Bus Line
+	2250 1400 2250 2900
+Wire Bus Line
+	3900 1300 3900 2100
 $EndSCHEMATC
